File: Hardware/Qwiic_VEML7700.brd (EAGLE design)
At the start: 25.4 x 25.4 mm, 46 parts, among them J1 Qwiic Right Angle, J2 PTH, J3 Qwiic Right Angle, U1 VEML7700-TT

Commit message: Add dimensions and measures
Parts:
- moved FRAME1 3.81 mm to (53.3, -8.89)
Other:
- board text added: "Dimensions in inches"
Changed lines of the file:
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@@
 <wire x1="25.4" y1="0" x2="0" y2="0" width="0.2032" layer="20"/>
 <text x="21.59" y="18.415" size="1.27" layer="16" font="vector" ratio="15" rot="MR0" align="center">x01</text>
-<dimension x1="0" y1="25.4" x2="0" y2="0" x3="-5.715003125" y3="12.7" textsize="1.778" textratio="15" layer="48" unit="inch" precision="1"/>
-<dimension x1="0" y1="25.4" x2="2.54" y2="22.86" x3="-2.771115625" y3="24.13" textsize="1.778" textratio="15" layer="48" dtype="vertical" unit="inch" precision="1"/>
-<dimension x1="25.4" y1="25.4" x2="0" y2="25.4" x3="12.7" y3="29.845003125" textsize="1.778" textratio="15" layer="48" unit="inch" precision="1"/>
-<dimension x1="25.4" y1="25.4" x2="22.86" y2="22.86" x3="24.13" y3="26.824078125" textsize="1.778" textratio="15" layer="48" dtype="horizontal" unit="inch" precision="1"/>
+<dimension x1="0" y1="25.4" x2="0" y2="0" x3="-5.715003125" y3="12.7" textsize="1.778" textratio="15" layer="47" unit="inch" precision="1"/>
+<dimension x1="0" y1="25.4" x2="2.54" y2="22.86" x3="-2.771115625" y3="24.13" textsize="1.778" textratio="15" layer="47" dtype="vertical" unit="inch" precision="1"/>
+<dimension x1="25.4" y1="25.4" x2="0" y2="25.4" x3="12.7" y3="29.845003125" textsize="1.778" textratio="15" layer="47" unit="inch" precision="1"/>
+<dimension x1="25.4" y1="25.4" x2="22.86" y2="22.86" x3="24.13" y3="26.824078125" textsize="1.778" textratio="15" layer="47" dtype="horizontal" unit="inch" precision="1"/>
 <text x="35.56" y="39.37" size="1.778" layer="51" font="vector" ratio="15" align="top-left">1.6mm PCB
 2-Layer
@@
 HASL Finish</text>
 <text x="80.3275" y="-7.239" size="1.778" layer="51" font="vector" ratio="15" align="top-left">Paul Clark</text>
+<text x="-2.54" y="-3.81" size="1.778" layer="47" ratio="15">Dimensions in inches</text>
 </plain>
 <attributes>
@@
 <attribute name="NAME" x="17.78" y="2.032" size="0.6096" layer="26" font="vector" ratio="20" rot="MR180"/>
 </element>
-<element name="FRAME1" library="SparkFun-Aesthetics" package="CREATIVE_COMMONS" value="FRAME-LETTER" x="49.53" y="-8.89" smashed="yes">
-<attribute name="DESIGNER" value="" x="49.53" y="-8.89" size="1.778" layer="27" display="off"/>
-<attribute name="REV" value="" x="49.53" y="-8.89" size="1.778" layer="27" display="off"/>
+<element name="FRAME1" library="SparkFun-Aesthetics" package="CREATIVE_COMMONS" value="FRAME-LETTER" x="53.34" y="-8.89" smashed="yes">
+<attribute name="DESIGNER" value="" x="53.34" y="-8.89" size="1.778" layer="27" display="off"/>
+<attribute name="REV" value="" x="53.34" y="-8.89" size="1.778" layer="27" display="off"/>
 </element>
 <element name="U$2" library="SparkX" package="SPARKX-MEDIUM" value="SPARKX-LOGO4" x="12.7" y="22.86" smashed="yes" rot="MR0"/>
